File: Poncho_rUVot/Poncho_rUVot.kicad_pcb (KiCad board)
At the start: 2 copper layers, 85.7 x 60.3 mm, 5 parts

Commit message: actualizacion
Connections:
- XA101 pad 1: +3.3VP -> +3V3
- XA101 pad 11: (no net) -> Net-(XA101-Pad11)
- XA101 pad 13: (no net) -> Net-(XA101-Pad13)
- XA101 pad 15: (no net) -> Net-(XA101-Pad15)
- XA101 pad 17: (no net) -> Net-(XA101-Pad17)
- XA101 pad 19: (no net) -> /SDA
- XA101 pad 21: (no net) -> /SCL
- XA101 pad 23: (no net) -> /RS232_RXD
- XA101 pad 25: (no net) -> /RS232_TXD
- XA101 pad 27: (no net) -> Net-(XA101-Pad27)
- XA101 pad 29: (no net) -> Net-(XA101-Pad29)
- XA101 pad 3: (no net) -> Net-(XA101-Pad3)
- XA101 pad 31: (no net) -> /T_COL1
- XA101 pad 33: (no net) -> Net-(XA101-Pad33)
- XA101 pad 34: (no net) -> Net-(XA101-Pad34)
- XA101 pad 35: (no net) -> /T_FIL3
- XA101 pad 36: (no net) -> Net-(XA101-Pad36)
- XA101 pad 37: (no net) -> Net-(XA101-Pad37)
- XA101 pad 39: (no net) -> Net-(XA101-Pad39)
- XA101 pad 42: +5V -> +5VP
- XA101 pad 43: GND -> GNDD
- XA101 pad 44: (no net) -> Net-(XA101-Pad44)
- XA101 pad 45: GND -> GNDD
- XA101 pad 46: (no net) -> Net-(XA101-Pad46)
- XA101 pad 47: GND -> GNDD
- XA101 pad 48: (no net) -> Net-(XA101-Pad48)
- XA101 pad 49: (no net) -> Net-(XA101-Pad49)
- XA101 pad 5: (no net) -> Net-(XA101-Pad5)
- XA101 pad 50: (no net) -> Net-(XA101-Pad50)
- XA101 pad 51: GND -> GNDD
- XA101 pad 52: (no net) -> Net-(XA101-Pad52)
- XA101 pad 53: GND -> GNDD
- XA101 pad 54: (no net) -> Net-(XA101-Pad54)
- XA101 pad 55: (no net) -> Net-(XA101-Pad55)
- XA101 pad 56: (no net) -> Net-(XA101-Pad56)
- XA101 pad 57: GND -> GNDD
- XA101 pad 58: (no net) -> Net-(XA101-Pad58)
- XA101 pad 59: GND -> GNDD
- XA101 pad 6: (no net) -> Net-(XA101-Pad6)
- XA101 pad 60: (no net) -> Net-(XA101-Pad60)
- XA101 pad 61: (no net) -> Net-(XA101-Pad61)
- XA101 pad 62: (no net) -> Net-(XA101-Pad62)
- XA101 pad 63: (no net) -> Net-(XA101-Pad63)
- XA101 pad 64: (no net) -> Net-(XA101-Pad64)
- XA101 pad 65: GND -> GNDD
- XA101 pad 66: (no net) -> Net-(XA101-Pad66)
- XA101 pad 67: GND -> GNDD
- XA101 pad 68: (no net) -> /LCD2
- XA101 pad 69: (no net) -> /GPIO0
- XA101 pad 70: (no net) -> /LCD1
- XA101 pad 71: (no net) -> /GPIO2
- XA101 pad 72: (no net) -> /GPIO1
- XA101 pad 73: (no net) -> /GPIO4
- XA101 pad 74: (no net) -> /GPIO3
- XA101 pad 75: (no net) -> /GPIO6
- XA101 pad 76: (no net) -> /GPIO5
- XA101 pad 77: GND -> GNDD
- XA101 pad 78: (no net) -> /GPIO7
- XA101 pad 79: GND -> GNDD
- XA101 pad 80: (no net) -> /GPIO8
- XA101 pad 9: (no net) -> Net-(XA101-Pad9)
