File: Poncho_rUVot/Poncho_rUVot.kicad_pcb (KiCad board)
At the start: 2 copper layers, 91.8 x 81 mm, 20 parts, among them J1 Screw_Terminal_01x03, K1 SANYOU_SRD_Form_C, P1 Conn_01x03, P2 Conn_01x03, P3 Conn_01x04, P4 Conn_01x03, P5 Conn_01x02, P6 Conn_01x02, P7 Conn_01x06, P8 Conn_01x04, P9 Conn_01x08, Q1 BC548, Q2 BC548

Commit message: Correcciones de detalles
Routing:
- added copper zone on B.Cu, net GND
Other:
- board text added: "Diseño simple faz. Sin requerimientos especiales. pistas: 0,6 mm y 0,8mm Margen: 1mm Distancia al borde: Documentaciòn superficial: HASL"
- board text removed: "Diseño simple faz. Sin requerimientos especiales. pistas: 0,6 mm y 0,8mm Margen: Distancia al borde: Documentaciòn superficial: HASL"
Changed lines of the file:
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@@
   )
   (setup
-    (last_trace_width 0.508)
+    (last_trace_width 0.381)
     (user_trace_width 0.508)
     (user_trace_width 0.6)
@@
     (user_trace_width 2)
     (trace_clearance 0.3)
-    (zone_clearance 0.508)
+    (zone_clearance 0.8)
     (zone_45_only no)
     (trace_min 0.2)
@@
   (gr_line (start 148.4 146) (end 121.92 146) (angle 90) (layer Edge.Cuts) (width 0.15))
   (gr_line (start 148.4 75) (end 148.4 146) (angle 90) (layer Edge.Cuts) (width 0.15))
-  (gr_text "Diseño simple faz.\nSin requerimientos especiales.\npistas: 0,6 mm y 0,8mm \nMargen: \nDistancia al borde: \nDocumentaciòn superficial: HASL\n" (at 191.75 33.25) (layer Dwgs.User)
+  (gr_text "Diseño simple faz.\nSin requerimientos especiales.\npistas: 0,6 mm y 0,8mm \nMargen:  1mm\nDistancia al borde: \nDocumentaciòn superficial: HASL\n" (at 191.75 33.25) (layer Dwgs.User)
     (effects (font (size 1.8 1.8) (thickness 0.4)) (justify left))
   )
@@
   (segment (start 76.103602 73.496398) (end 77 72.6) (width 0.8) (layer B.Cu) (net 2))
   (segment (start 76.103602 78.103602) (end 76.103602 73.496398) (width 0.8) (layer B.Cu) (net 2))
-  (segment (start 99.54 73.94) (end 99.54 74.8) (width 0.381) (layer B.Cu) (net 48))
   (segment (start 77 72.6) (end 80.6 72.6) (width 0.8) (layer B.Cu) (net 2))
   (segment (start 81.54 73.54) (end 81.54 74.8) (width 0.8) (layer B.Cu) (net 2))
@@
   (segment (start 125.95 142.75) (end 125.2 142) (width 0.508) (layer B.Cu) (net 47))
   (segment (start 133.25 142.75) (end 125.95 142.75) (width 0.508) (layer B.Cu) (net 47))
+  (segment (start 99.54 73.94) (end 99.54 74.8) (width 0.381) (layer B.Cu) (net 48))
   (segment (start 58.72 67.92) (end 60.2 66.44) (width 0.6) (layer B.Cu) (net 48))
   (segment (start 58.72 127.6) (end 58.72 67.92) (width 0.6) (layer B.Cu) (net 48))
@@
   (segment (start 81.52384 104.97312) (end 81.72704 105.17632) (width 0.381) (layer B.Cu) (net 65))
   (segment (start 81.52384 97.8027) (end 81.52384 104.97312) (width 0.6) (layer B.Cu) (net 65))
+  (zone (net 2) (net_name GND) (layer B.Cu) (hatch edge 0.508)
+    (connect_pads (clearance 0.8))
+    (min_thickness 0.6)
+    (fill yes (arc_segments 32) (thermal_gap 0.65) (thermal_bridge_width 0.65))
+    (polygon
+      (pts
+        (xy 150 147) (xy 55 147) (xy 55 64) (xy 150 64)
+      )
+    )
+  )
 )

Commit message: Correcciones sugeridas
Parts:
- added G***: LOGO, footprint:Logo_Poncho, F.Cu at (98.0, 84.0)
- added REF**: OSHW-Logo2_7.3x6mm_SilkScreen, Symbol:OSHW-Logo2_7.3x6mm_SilkScreen, F.Cu at (108.0, 85.0)
Other:
- outline, holes or cut-outs redrawn
- board text added: "Detalles de diseño"
- board text added: "Diseño simple faz. Sin requerimientos especiales. Unidades: metric. Pistas: 0,6 mm y 0,8mm. Margen: 1mm. Distancia de track al borde: >4mm. Documentaciòn superficial: HASL."
- board text added: "Motor"
- board text added: "Poncho rUVot - Sergio Alberino Industria Argentina"
- board text removed: "Diseño simple faz. Sin requerimientos especiales. pistas: 0,6 mm y 0,8mm Margen: 1mm Distancia al borde: Documentaciòn superficial: HASL"
- board text removed: "Poncho rUVot - Sergio Alberino"
- board text removed: "STACK-UP"

Commit message: Correcciones de PCB sugeridas
Parts:
- removed G***: LOGO, footprint:Logo_Poncho
- removed REF**: OSHW-Logo2_7.3x6mm_SilkScreen, Symbol:OSHW-Logo2_7.3x6mm_SilkScreen
- added H1: MountingHole, MountingHole:MountingHole_2.5mm, F.Cu at (143.6, 79.4)
- Q1, Q2: footprint Package_TO_SOT_THT:TO-92L -> Package_TO_SOT_THT:TO-92L_Wide
- moved R4 4.95 mm to (94.2, 103.4)
- moved D2 4.40 mm to (94.2, 109.4)
- moved R2 2.09 mm to (80.0, 104.0)
- moved P1 1.80 mm to (67.0, 74.8)
- moved R1 1.68 mm to (87.0, 104.0)
- moved Q2 0.79 mm to (82.0, 96.5)
- moved Q1 0.53 mm to (90.0, 96.6)
Routing:
- net +5V: track 179.1 -> 192.5 mm, vias 2 -> 4
- net Net-(D1-Pad2): track 23.0 -> 31.5 mm
- net /LCD1: track 26.8 -> 22.7 mm
- net /GPIO4: track 95.5 -> 91.7 mm
- net /GPIO2: track 86.0 -> 82.7 mm
- net /LCD2: track 17.9 -> 14.6 mm
- net Net-(Q1-Pad2): track 7.44 -> 5.09 mm
- net Net-(Q2-Pad2): track 7.46 -> 5.15 mm
- net /T_FIL3: track 13.3 -> 15.5 mm
- net /GPIO0: track 67.6 -> 65.8 mm
- net Net-(BZ1-Pad2): track 7.44 -> 8.55 mm
- net Net-(D2-Pad2): track 4.03 -> 3.46 mm
Other:
- net class Default: clearance 0.3 -> 0.5
- rule trace_clearance: 0.3 -> 0.5
- board text added: "Detalles de fabricación"
- board text added: "Diseño simple faz. Sin requerimientos especiales. Documentación superficial: HASL. Fabricación casera"
- board text added: "Diseño simple faz. Sin requerimientos especiales. Unidades: metric. Grilla: 1mm. Pistas: 0,6 mm y 0,8mm. Margen: 1mm. Distancia de track al borde: >4mm."
- board text removed: "Diseño simple faz. Sin requerimientos especiales. Unidades: metric. Pistas: 0,6 mm y 0,8mm. Margen: 1mm. Distancia de track al borde: >4mm. Documentaciòn superficial: HASL."
