File: Poncho_rUVot/_autosave-Poncho_rUVot.sch (KiCad schematic (older format))
At the start: 20 parts, among them J1 Screw_Terminal_01x03, K1 SANYOU_SRD_Form_C, P1 Conn_01x03, P2 Conn_01x03, P3 Conn_01x04, P4 Conn_01x03, P5 Conn_01x02, P6 Conn_01x02, P7 Conn_01x06, P8 Conn_01x04, P9 Conn_01x08, Q1 BC548, Q2 BC548

Commit message: Correcciones de PCB sugeridas
Parts:
- added H1: MountingHole, MountingHole:MountingHole_2.5mm, symbol Mechanical:MountingHole
- Q1, Q2: footprint Package_TO_SOT_THT:TO-92L -> Package_TO_SOT_THT:TO-92L_Wide
Changed lines of the file:
@@
 F 0 "Q2" H 10541 5596 50  0000 L CNN
 F 1 "BC548" H 10541 5505 50  0000 L CNN
-F 2 "Package_TO_SOT_THT:TO-92L" H 10550 5475 50  0001 L CIN
+F 2 "Package_TO_SOT_THT:TO-92L_Wide" H 10550 5475 50  0001 L CIN
 F 3 "https://www.onsemi.com/pub/Collateral/BC550-D.pdf" H 10350 5550 50  0001 L CNN
 	1    10350 5550
@@
 F 0 "Q1" H 7741 5596 50  0000 L CNN
 F 1 "BC548" H 7741 5505 50  0000 L CNN
-F 2 "Package_TO_SOT_THT:TO-92L" H 7750 5475 50  0001 L CIN
+F 2 "Package_TO_SOT_THT:TO-92L_Wide" H 7750 5475 50  0001 L CIN
 F 3 "https://www.onsemi.com/pub/Collateral/BC550-D.pdf" H 7550 5550 50  0001 L CNN
 	1    7550 5550
@@
 	1    0    0    -1
 $EndComp
+$Comp
+L Mechanical:MountingHole H1
+U 1 1 608D861A
+P 4200 6000
+F 0 "H1" H 4300 6046 50  0000 L CNN
+F 1 "MountingHole" H 4300 5955 50  0000 L CNN
+F 2 "MountingHole:MountingHole_2.5mm" H 4200 6000 50  0001 C CNN
+F 3 "~" H 4200 6000 50  0001 C CNN
+	1    4200 6000
+	1    0    0    -1
+$EndComp
